File: LuciCameraLettoRoma/LuciCameraLettoRoma.kicad_pcb (KiCad board)
At the start: 2 copper layers, 67.3 x 114.7 mm, 82 parts, among them J1 Screw_Terminal_01x04, J2 Screw_Terminal_01x04, J3 Screw_Terminal_01x04, K1 RT42xAxx, K2 RT42xAxx, K3 RT42xAxx, K4 RT42xAxx, K5 RT42xAxx, Q1 IRLML0030, Q2 IRLML0030, Q3 IRLML0030, Q4 IRLML0030, Q5 IRLML0030, Q6 IRLML0030, Q7 IRLML0030, Q8 IRLML0030, U1 ATmega328-PU, U2 CRE1S0505S3C, U3 AQY214EH, U4 AQY214EH, U5 AQY214EH, Y1 16MHz

Commit message: Add files via upload
Parts:
- removed  AltaTensione: Symbol_HighVoltage_Type2_CopperTop_VerySmall, Symbol:Symbol_HighVoltage_Type2_CopperTop_VerySmall
- removed the J1 at (94.7, 72.8)
- removed Pul.2, Pul.3: Screw_Terminal_01x02, Connector_Phoenix_MC_HighVoltage:PhoenixContact_MCV_1,5_2-G-5.08_1x02_P5.08mm_Vertical
- added AltaTensione: , Symbol:Symbol_HighVoltage_Type2_CopperTop_VerySmall, B.Cu at (108.0, 100.2)
- added AltaTensione: , Symbol:Symbol_HighVoltage_Type2_CopperTop_VerySmall, B.Cu at (107.9, 67.5)
- added AltaTensione: , Symbol:Symbol_HighVoltage_Type2_CopperTop_VerySmall, B.Cu at (118.9, 84.0)
- added AltaTensione: , Symbol:Symbol_HighVoltage_Type2_CopperTop_VerySmall, B.Cu at (118.7, 67.7)
- added AltaTensione: , Symbol:Symbol_HighVoltage_Type2_CopperTop_VerySmall, B.Cu at (108.1, 84.0)
- added AltaTensione: , Symbol:Symbol_HighVoltage_Type2_CopperTop_VerySmall, B.Cu at (118.7, 117.4)
- added AltaTensione: , Symbol:Symbol_HighVoltage_Type2_CopperTop_VerySmall, B.Cu at (118.6, 100.2)
- added AltaTensione: , Symbol:Symbol_HighVoltage_Type2_CopperTop_VerySmall, B.Cu at (110.6, 134.4)
- added AltaTensione: , Symbol:Symbol_HighVoltage_Type2_CopperTop_VerySmall, B.Cu at (100.2, 115.8)
- Alta Tensione: renamed from AltaTensione; value Symbol_HighVoltage_Type2_CopperTop_VerySmall -> (none)
- Analog-0-1: renamed from Analog-0-2; value Conn_01x04_Male -> (none)
- Analog-3-1: renamed from Analog-3-5; value Conn_01x04_Male -> (none)
- D1: renamed from D2; value LED -> P1
- D2: renamed from D7; value LED -> P1
- D3: renamed from D8; value LED -> P2
- D4: renamed from D9; value LED -> P3
- D5: renamed from D1; value LED -> K1
- D6: renamed from D3; value LED -> K2
- D7: renamed from D4; value LED -> K3
- D8: renamed from D5; value LED -> K4
- D9: renamed from D6; value LED -> K5
- J1: renamed from Pul.1; value Screw_Terminal_01x02 -> (none); footprint Connector_Phoenix_MC_HighVoltage:PhoenixContact_MCV_1,5_2-G-5.08_1x02_P5.08mm_Vertical -> Connector_PinSocket_2.54mm:PinSocket_1x04_P2.54mm_Horizontal
- J2: value Screw_Terminal_01x04 -> (none); footprint Connector_Phoenix_MC:PhoenixContact_MC_1,5_4-G-3.81_1x04_P3.81mm_Horizontal -> Connector_PinSocket_2.54mm:PinSocket_1x10_P2.54mm_Horizontal
- J3: value Screw_Terminal_01x04 -> (none); footprint Connector_Phoenix_MC:PhoenixContact_MC_1,5_4-G-3.81_1x04_P3.81mm_Horizontal -> Connector_PinSocket_2.54mm:PinSocket_1x02_P2.54mm_Horizontal
- K1, K2, K3, K4, K5: value RT42xAxx -> (none); footprint Relay_THT:Relay_DPDT_Schrack-RT2-FormC_RM5mm -> Relay_THT:Relay_SPDT_SANYOU_SRD_Series_Form_C
- PS1: value RAC04-05SGA -> HLK-5M05; footprint Converter_ACDC:AC-DC 240-5V 0.7A -> Converter_ACDC:CONV_HLK-5M05
- Power-Reset1: value Conn_01x04_Male -> (none)
- Prog-RS1: renamed from Prog-RS232; value Conn_01x04_Male -> (none)
- Q1: renamed from Q6; value IRLML0030 -> (none)
- Q3: renamed from Q8; value IRLML0030 -> (none); moved to F.Cu
- R20: renamed from R1; moved to F.Cu
- SPI+1: value Conn_01x06_Male -> (none)
- SlowReset1: value Jumper_2_Open -> (none)
- U2: renamed from U3; value AQY214EH -> (none)
- U3: renamed from U4; value AQY214EH -> (none)
- Vite1, Vite2, Vite3, Vite4: value MountingHole_3.5mm_Pad_Via -> (none)
- moved Alta Tensione 63.7 mm to (97.4, 98.6), turned to -90 degrees
- moved J2 35.2 mm to (100.7, 67.2), turned to 0 degrees
- moved K5 27.4 mm to (99.1, 124.0), turned to 90 degrees
- moved REFht1 22.4 mm to (96.0, 128.9), turned to 0 degrees
- moved Logo1 19.8 mm to (94.5, 149.4), turned to 90 degrees
- moved Wast01 15.0 mm to (102.7, 58.2)
- moved L1 13.7 mm to (147.7, 94.7), turned to -90 degrees
- moved Wast02 13.5 mm to (104.4, 60.5)
- moved D2 11.0 mm to (149.6, 131.6)
- moved C7 10.9 mm to (140.3, 59.6)
- moved R20 8.47 mm to (147.8, 68.5), turned to 90 degrees
- moved J3 8.39 mm to (100.5, 135.4), turned to 0 degrees
- moved Analog-0-1 7.88 mm to (152.0, 87.4), turned to 180 degrees
- moved C2 7.13 mm to (147.7, 89.7), turned to -90 degrees
- moved J1 7.08 mm to (149.5, 145.7), turned to 180 degrees
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- renumbered C7 to C1, C5 to C2, C1 to C3, C2 to C4, C3 to C5, C4 to C6, C6 to C7, L2 to L1, L1 to L2, Q7 to Q2, Q1 to Q4, Q2 to Q5, Q3 to Q6, Q4 to Q7, Q5 to Q8, R2 to R1, R9 to R10, R10 to R11, R11 to R12, R12 to R13, R13 to R14, R14 to R15, R15 to R16, R16 to R17, R17 to R18, R3 to R19, R18 to R2, R4 to R3, R5 to R4, R19 to R5, R20 to R7, R7 to R8, R8 to R9, REF** to REFht1, U2 to U1, U5 to U4, U1 to U5
Connections:
- net /Luci Camera Letto Roma CPU/-1*Reset renamed /Luci Camera Letto Roma CPU/Reset
- net /Luci Camera Letto Roma CPU/IO0-RS232-RX renamed /Luci Camera Letto Roma CPU/Rx
- net /Luci Camera Letto Roma CPU/IO1-RS232-TX renamed /Luci Camera Letto Roma CPU/Tx
- net /Luci Camera Letto Roma CPU/IO2 renamed /Luci Camera Letto Roma - Rele/Rele-IO2
- net /Luci Camera Letto Roma CPU/IO3 renamed /Luci Camera Letto Roma - Rele/Rele-IO3
- net /Luci Camera Letto Roma CPU/IO4 renamed /Luci Camera Letto Roma - Rele/Rele-IO4
- net /Luci Camera Letto Roma CPU/IO5 renamed /Luci Camera Letto Roma - Rele/Rele-IO5
- net /Luci Camera Letto Roma CPU/IO6 renamed /Luci Camera Letto Roma - Rele/Rele-IO6
- net /Luci Camera Letto Roma CPU/IO7 renamed /Luci Camera Letto Roma - Input/Pulsante1-IO
- net /Luci Camera Letto Roma CPU/IO8 renamed /Luci Camera Letto Roma - Input/Pulsante2-IO
- net /Luci Camera Letto Roma CPU/IO9 renamed /Luci Camera Letto Roma - Input/Pusante3-IO
- Analog-3-1 pad 2: /Luci Camera Letto Roma CPU/A3 -> /Luci Camera Letto Roma CPU/A5-I2C-SCL
- Analog-3-1 pad 4: /Luci Camera Letto Roma CPU/A5-I2C-SCL -> /Luci Camera Letto Roma CPU/A3
- D5 pad 1: Net-(D1-Pad1) -> Net-(D5-Pad1)
- D6 pad 1: Net-(D3-Pad1) (its old number) -> Net-(D6-Pad1)
- D7 pad 1: Net-(D4-Pad1) (its old number) -> Net-(D7-Pad1)
- D8 pad 1: Net-(D5-Pad1) -> Net-(D8-Pad1)
- D9 pad 1: Net-(D6-Pad1) -> Net-(D9-Pad1)
- PS1 pad 1: Net-(J3-Pad4) -> Net-(J3-Pad2)
- PS1 pad 2: Net-(J3-Pad3) -> Net-(J3-Pad1)
- PS1 pad 3: Net-(PS1-Pad3) -> GND
- PS1 pad 4: GND -> +5V
- Power-Reset1 pad 3: Net-(Power-Reset1-Pad3) -> unconnected-(Power-Reset1-Pad3)
- Q4 pad 3: Net-(D1-Pad1) -> Net-(D5-Pad1)
- Q5 pad 3: Net-(D3-Pad1) (its old number) -> Net-(D6-Pad1)
- Q6 pad 3: Net-(D4-Pad1) (its old number) -> Net-(D7-Pad1)
- Q7 pad 3: Net-(D5-Pad1) -> Net-(D8-Pad1)
- Q8 pad 3: Net-(D6-Pad1) -> Net-(D9-Pad1)
- R11 pad 2: Net-(J6-Pad2) -> Net-(J1-Pad4)
- R12 pad 2: Net-(J6-Pad2) -> Net-(J1-Pad4)
- R8 pad 2: Net-(J5-Pad2) -> Net-(J1-Pad3)
- R9 pad 2: Net-(J5-Pad2) -> Net-(J1-Pad3)
- U3 pad 1: Net-(J5-Pad2) -> Net-(J1-Pad3)
- U4 pad 1: Net-(J6-Pad2) -> Net-(J1-Pad4)
- U5 pad 21: Net-(U1-Pad21) -> unconnected-(U5-Pad21)
Routing:
- net +5V: track 230.1 -> 308.3 mm, vias 0 -> 1
- net Net-(K4-Pad1): track 0.00 -> 46.7 mm
- net GND: track 369.3 -> 324.4 mm, vias 4 -> 0
- net Net-(D9-Pad1): track 0.00 -> 37.2 mm, vias 0 -> 1
- net Net-(K3-Pad1): track 0.00 -> 35.5 mm
- net Net-(J2-Pad10): track 0.00 -> 34.6 mm
- net GNDD: track 88.4 -> 55.7 mm
- net Net-(K4-Pad3): track 0.00 -> 32.3 mm
- net Net-(D7-Pad1): track 0.00 -> 26.6 mm
- net Net-(J2-Pad9): track 0.00 -> 25.4 mm
- net Net-(J2-Pad4): track 8.50 -> 29.3 mm
- net Net-(K3-Pad3): track 0.00 -> 20.7 mm
- net Net-(J2-Pad2): track 6.94 -> 26.5 mm
- net Net-(J1-Pad4): track 8.32 -> 27.8 mm
- net Net-(J3-Pad3): track 18.9 -> 0.00 mm
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- removed copper zone on B.Cu, net GNDD
- removed copper zone on F.Cu, net GNDD
Other:
- board size 67.3 x 114.7 mm -> 67.3 x 114.6 mm
- net class 240VAC removed
- net class Default removed
- net class Power removed
